File: mercury/mercury.kicad_sch (KiCad schematic)
At the start: 65 parts, among them J1 Right_Motor_Connector, J2 Left_Motor_Connector, Q1 NMOS, Q2 NMOS, Q3 NMOS, Q4 TEFT4300, Q5 TEFT4300, Q6 TEFT4300, Q7 TEFT4300, U1 ZXMHC3F381N8TC, U2 UCC27524ADR, U3 UCC27524ADR, U4 ZXMHC3F381N8TC, U5 MCP1700, U6 TPS73633DBV, U7 TPS76850QDR, U8 CP2102N-Axx-xQFN28, U9 ESP32-S3-WROOM-1U-N16R8

Commit message: added more to pcb, esp32, gyro, usbc
Parts:
- added BT1: Battery, symbol Device:Battery_Cell
- added C23, C25, C29, C31: 0.1uF, symbol Device:C
- added C24, C27, C28: 2.2uF, symbol Device:C
- added C26: 1uF, symbol Device:C
- added C30: 10nF, symbol Device:C
- added D5, D6: SFH4545, MM_Library:Emitter, symbol bloo-rescue:IRL81A-LED-mouse_v2-rescue
- added D7: SP0503BAHT, Package_TO_SOT_SMD:SOT-143, symbol Mercury_Symbols:SP0503BAHT
- added J3: USB_C_Receptacle_USB2.0, Connector_USB:USB_C_Receptacle_GCT_USB4085, symbol Connector:USB_C_Receptacle_USB2.0
- added Q10, Q11: TEFT4300, MM_Library:Emitter, symbol bloo-rescue:Q_Photo_NPN-Device-mouse_v2-rescue
- added Q8, Q9: NMOS, symbol Simulation_SPICE:NMOS
- added R16, R19, R21: 10k, symbol Device:R_US
- added R17, R18: 5.1k, symbol Device:R_US
- added R20: 20k, symbol Device:R_US
- added R22, R24: 47k, symbol Device:R_US
- added R23, R25: 10, symbol Device:R_US
- added R26, R27: 1.8k, symbol Device:R_US
- added SW1, SW2: SW_Push, symbol Switch:SW_Push
- added U10: MPU-6500, footprint:QFN24_3X3X0P9_IVS, symbol Mercury_Symbols:MPU-6500
- R12, R13, R14, R15: footprint OptoDevice:R_LDR_D6.4mm_P3.4mm_Vertical -> (none)
- U1, U4: footprint SOIC_81N8TC_DIO -> footprint:SOIC_81N8TC_DIO
- U2, U3, U7: footprint D8_TEX -> footprint:D8_TEX
- U9: footprint (none) -> footprint:ESP32­S3­WROOM­1U_EXP
Connections:
- net 3.3VA_RECV is gone; now on net RECV_3.3VA: C5.1, U5.3 (VO)
- net FL_EMITTER is gone; now on net FL_EMIT: Q1.2 (G), R2.1
- net FR_EMITTER is gone; now on net FR_EMIT: Q2.2 (G), R4.1
- net VBUS is gone; now on net 5V: R13.1
- net 3.3V: now also R19.1
- net 5V: now also D5.2 (A), D6.2 (A), D7.2 (K), J3.A4 (VBUS), J3.A9 (VBUS), J3.B4 (VBUS), J3.B9 (VBUS)
- net AGND: now also C28.2, C29.2, C30.1, C31.1, U10.18 (GND), U10.20 (RESV), U10.25; no longer C1.2, C2.2, C3.2, C4.2, R10.2, R7.2, R8.2, R9.2
- net FL_RECV: now also U9.10 (IO17)
- net FR_RECV: now also U9.13 (IO19)
- net GND: now also BT1.2 (-), C23.1, C25.1, C26.2, D7.1 (A), J3.A1 (GND), J3.A12 (GND), J3.B1 (GND), J3.B12 (GND), J3.S1 (SHIELD), Q8.3 (S), Q9.3 (S), R16.2, R17.2, R18.2, R21.2, R22.2, R24.2, SW1.1, SW2.1
- net MR_ENC_A: now also U9.22 (IO14); no longer U9.23 (IO21)
- net MR_ENC_B: now also U9.21 (IO13); no longer U9.24 (IO47)
- net MR_PWMA: now also U9.24 (IO47); no longer U9.21 (IO13)
- net MR_PWMB: now also U9.23 (IO21); no longer U9.22 (IO14)
- net USB_D+: now also U8.4 (D+), D7.4 (K), J3.A6 (D+), J3.B6 (D+); no longer U9.14 (IO20)
- net USB_D-: now also U8.5 (D-), D7.3 (K), J3.A7 (D-), J3.B7 (D-); no longer U9.13 (IO19)
- net V_BATTERY: now also S1.2, S1.3, R20.1; no longer U4.7 (P1S/P2S)
- net DL_RECV: now reaches U9.11 (IO18)
- net DR_RECV: now reaches U9.12 (IO8)
- net BOOT: now reaches U9.27 (IO0)
- net BOOT: now also C25.2, C26.1, R19.2, SW2.2
- net DIAG_EMIT: now reaches U9.33 (IO40)
- net FL_EMIT: now reaches U9.34 (IO41)
- net FR_EMIT: now reaches U9.35 (IO42)
- net BATT_DIV: now reaches U9.8 (IO15)
- net BATT_DIV: now also R20.2, R21.1
- net SL_RECV: now reaches U9.9 (IO16)
- net at U8.11 (~{SUSPEND}): now also R16.1
- net at S1.1: now also BT1.1 (+)
- net 3.3VA renamed RECV_3.3VA
- net RECV_3.3VA: now also C24.1, C27.1, Q10.1 (C), Q11.1 (C); no longer C14.1, L4.2
- net AGND_RECV renamed RECV_GND
- net RECV_GND: now also C1.2, C2.2, C3.2, C4.2, R10.2, R7.2, R8.2, R9.2, C24.2, C27.2, R26.2, R27.2
- net DIAGONAL_EMMITER renamed D_EMIT
- net DTR: no longer names the net of U8.28 (~{DTR})
- net EN renamed RST
- net RST: now also C23.2, SW1.2
- net RTS: no longer names the net of U8.24 (~{RTS})
- net U0RTX renamed UART_RX
- net U0TXD renamed UART_TX
- new net: C31.2, U10.10 (REGOUT)
- new net: J3.A5 (CC1), R18.1
- new net: J3.B5 (CC2), R17.1
- new net: Q9.1 (D), R25.2
- new net: D5.1 (K), R23.1
- new net: Q8.1 (D), R23.2
- new net: D6.1 (K), R25.1
- new net A3.3V: C14.1, C28.1, C29.1, C30.2, L4.2, U10.13 (VDD), U10.8 (VDDIO)
- new net B_BATTERY: U4.7 (P1S/P2S)
- new net FSYNC: U10.11 (FSYNC)
- new net INT: U10.12 (INT)
- new net NCS: U10.22 (nCS)
- new net SCLK: U10.23 (SCL/SCLK)
- new net SDI: U10.24 (SDA/SDI)
- new net SDO: U10.9 (SDO/ADO)
- new net SR_EMIT: Q8.2 (G), Q9.2 (G), R22.1, R24.1
- new net SR_RECV: Q10.2 (E), R26.1, U9.14 (IO20)
- new net Sl_RECV: Q11.2 (E), R27.1
- no-connect marks 21 -> 27
Other:
- moved on the sheet: C1, C10, C11, C12, C13, C14, C15, C16, C17, C18, C19, C2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

Commit message: first completerouting of PCB
Parts:
- removed BT1: Battery, symbol Device:Battery_Cell
- removed C16, C17: 100uF, symbol Device:C
- removed C18: 0.1uF, symbol Device:C
- removed J1: Right_Motor_Connector, symbol Connector:Conn_01x06_Socket
- removed J2: Left_Motor_Connector, symbol Connector:Conn_01x06_Socket
- removed L4, L5: 10uH, symbol Device:L
- removed S1: EG1218, MM_Library:MM Switch, symbol bloo-rescue:EG1218-dk_Slide-Switches-mouse-rescue
- removed U7: TPS76850QDR, footprint:D8_TEX, symbol Mercury_Symbols:TPS76850QDR
- removed U8: CP2102N-Axx-xQFN28, Package_DFN_QFN:SiliconLabs_QFN-20-1EP_3x3mm_P0.5mm, symbol Interface_USB:CP2102N-Axx-xQFN28
- added C35, C40, C41, C48, C49, C50: 10uF, Capacitor_SMD:C_0603_1608Metric_Pad1.08x0.95mm_HandSolder, symbol Device:C
- added C36, C38: 100nF, Capacitor_SMD:C_0603_1608Metric_Pad1.08x0.95mm_HandSolder, symbol Device:C
- added C37, C39: 1uF, Capacitor_SMD:C_0603_1608Metric_Pad1.08x0.95mm_HandSolder, symbol Device:C
- added C42: 10uF (Tantalum), Capacitor_SMD:C_0603_1608Metric_Pad1.08x0.95mm_HandSolder, symbol Device:C
- added C43: 470pF, Capacitor_SMD:C_0603_1608Metric_Pad1.08x0.95mm_HandSolder, symbol Device:C
- added C44: 47uF, Capacitor_SMD:C_0603_1608Metric_Pad1.08x0.95mm_HandSolder, symbol Device:C
- added C45: 0.1uF, Capacitor_SMD:C_0603_1608Metric_Pad1.08x0.95mm_HandSolder, symbol Device:C
- added C46, C47: 100uF, Capacitor_SMD:C_0603_1608Metric_Pad1.08x0.95mm_HandSolder, symbol Device:C
- added D8: 1N5819HW-7-F, footprint:1N5819HW-7-F_DIO, symbol Diode:1N5819
- added D9: SL_EMIT, footprint:Emitter, symbol bloo-rescue:IRL81A-LED-mouse_v2-rescue
- added IC1: AS5600-ML, footprint:SOIC127P600X175-8N, symbol Mercury_Symbols:AS5600-ASOT
- added IC2: AS5600-MR, footprint:SOIC127P600X175-8N, symbol Mercury_Symbols:AS5600-ASOT
- added J1: Battery, Connector_PinSocket_2.54mm:PinSocket_1x02_P2.54mm_Vertical, symbol Connector:Conn_01x02_Socket
- added J2: UART, Connector_PinHeader_2.54mm:PinHeader_1x04_P2.54mm_Vertical, symbol Connector:Conn_01x04_Socket
- added J4, J5: Conn_01x02_Socket, Connector_PinSocket_2.54mm:PinSocket_1x02_P2.54mm_Vertical, symbol Connector:Conn_01x02_Socket
- added J6: Encoder_L, Connector_PinHeader_2.54mm:PinHeader_1x04_P2.54mm_Vertical, symbol Connector:Conn_01x04_Socket
- added J7: Encoder_R, Connector_PinHeader_2.54mm:PinHeader_1x04_P2.54mm_Vertical, symbol Connector:Conn_01x04_Socket
- added Q12: NMOS, footprint:SOT-23, symbol Simulation_SPICE:NMOS
- added R28: 10k, Resistor_SMD:R_0603_1608Metric_Pad0.98x0.95mm_HandSolder, symbol Device:R_US
- added R31, R32, R33, R34, R35, R36: 4.7k, Resistor_SMD:R_0603_1608Metric_Pad0.98x0.95mm_HandSolder, symbol Device:R_US
- added R40: 47k, Resistor_SMD:R_0603_1608Metric_Pad0.98x0.95mm_HandSolder, symbol Device:R_US
- added R45: 223k, Resistor_SMD:R_0603_1608Metric_Pad0.98x0.95mm_HandSolder, symbol Device:R_US
- added R46: 115k, Resistor_SMD:R_0603_1608Metric_Pad0.98x0.95mm_HandSolder, symbol Device:R_US
- added SW3, SW4: SW_Push, footprint:SW_SPST_REED_CT05-XXXX-G1, symbol Switch:SW_Push
- added U11, U7: ~, footprint:HTSOP-J8_ROM, symbol Mercury_Symbols:BD60FC0WEFJ-E2
- added U12: LMZ10501SILR, footprint:SIL0008A, symbol LMZ10501SILR:LMZ10501SILR
- added U8: LM1085-5.0, footprint:5V Voltage Reg, symbol Regulator_Linear:LM1085-5.0
- C1, C10, C11, C12, C13, C15, C19, C2, C20, C21, C23, C24, C25, C27, C28, C29, C3, C30, C31, C4, C5, C6, C7, C8, C9: footprint (none) -> Capacitor_SMD:C_0603_1608Metric_Pad1.08x0.95mm_HandSolder
- C14: value 2.2uF -> 0.1uF; footprint (none) -> Capacitor_SMD:C_0603_1608Metric_Pad1.08x0.95mm_HandSolder
- C22, C26: value 1uF -> 0.1uF; footprint (none) -> Capacitor_SMD:C_0603_1608Metric_Pad1.08x0.95mm_HandSolder
- D1: value SFH4545 -> FL_EMIT; footprint MM_Library:Emitter -> footprint:Emitter
- D2: value SFH4545 -> FR_EMIT; footprint MM_Library:Emitter -> footprint:Emitter
- D3: value SFH4545 -> R_EMIT; footprint MM_Library:Emitter -> footprint:Emitter
- D4: footprint (none) -> LED_SMD:LED_0805_2012Metric_Pad1.15x1.40mm_HandSolder
- D5: value SFH4545 -> L_EMIT; footprint MM_Library:Emitter -> footprint:Emitter
- D6: value SFH4545 -> SR_EMIT; footprint MM_Library:Emitter -> footprint:Emitter
- L1, L2, L3: footprint (none) -> Inductor_SMD:L_0603_1608Metric_Pad1.05x0.95mm_HandSolder
- Q1, Q2, Q3, Q8, Q9: footprint (none) -> footprint:SOT-23
- Q10: value TEFT4300 -> SR_RECV; footprint MM_Library:Emitter -> footprint:IR_Receiver_Mirrored
- Q11: value TEFT4300 -> SL_RECV; footprint MM_Library:Emitter -> footprint:IR_Reciever
- Q4: value TEFT4300 -> FR_RECV; footprint MM_Library:Emitter -> footprint:IR_Reciever
- Q5: value TEFT4300 -> FL_RECV; footprint MM_Library:Emitter -> footprint:IR_Receiver_Mirrored
- Q6: value TEFT4300 -> R_RECV; footprint MM_Library:Emitter -> footprint:IR_Receiver_Mirrored
- Q7: value TEFT4300 -> L_RECV; footprint MM_Library:Emitter -> footprint:IR_Reciever
- R1, R10, R11, R12, R16, R17, R18, R19, R2, R20, R21, R22, R23, R24, R25, R26, R27, R3, R4, R5, R6, R7, R8, R9: footprint (none) -> Resistor_SMD:R_0603_1608Metric_Pad0.98x0.95mm_HandSolder
- R13: value 22.1k -> 47k; footprint (none) -> Resistor_SMD:R_0603_1608Metric_Pad0.98x0.95mm_HandSolder
- R14: value 1k -> 10; footprint (none) -> Resistor_SMD:R_0603_1608Metric_Pad0.98x0.95mm_HandSolder
- R15: value 47.5 -> 10k; footprint (none) -> Resistor_SMD:R_0603_1608Metric_Pad0.98x0.95mm_HandSolder
- SW1, SW2: footprint (none) -> footprint:SW_SPST_REED_CT05-XXXX-G1
Connections:
- net AGND is gone; now on net GND: C14.2, C28.2, C29.2, C30.1, C31.1, U10.18 (GND), U10.20 (RESV), U10.25
- net FSYNC is gone; now on net GND: U10.11 (FSYNC)
- net L_RECV is gone; now on net DL_RECV: Q7.2 (E), R10.1
- net ML_ENC_B is gone; now on net SR_EMIT: U9.17 (IO9)
- net MR_ENC_A is gone; now on net DL_RECV: U9.22 (IO14)
- net MR_ENC_B is gone; now on net SL_RECV: U9.21 (IO13)
- net NCS is gone; now on net 3.3V: U10.22 (nCS)
- net R_RECV is gone; now on net DR_RECV: Q6.2 (E), R9.1
- net SCLK is gone; now on net SCL_1: U10.23 (SCL/SCLK)
- net SDO is gone; now on net GND: U10.9 (SDO/ADO)
- net Sl_RECV is gone; now on net SL_RECV: Q11.2 (E), R27.1
- net 3.3V: now also C28.1, C29.1, C30.2, R15.1, R16.1, R19.2, U10.13 (VDD), U10.8 (VDDIO), J6.1 (Pin_1), J7.1 (Pin_1), R28.2; no longer R14.1, R19.1
- net 5V: now also C26.2, C36.1, C38.1, C41.1, C42.2, C46.2, D8.1 (K), IC1.1 (VDD5V), IC2.1 (VDD5V), J2.1 (Pin_1), R32.2, R33.2, R34.2, R35.2, R36.2, U11.5 (EN), U12.7 (VIN), U7.5 (EN), U8.2 (VO); no longer D1.2 (A), D2.2 (A), D3.2 (A), D5.2 (A), D6.2 (A), D7.2 (K), J3.A4 (VBUS), J3.A9 (VBUS), J3.B4 (VBUS), J3.B9 (VBUS), R13.1
- net BATT_DIV: now also R20.1, U9.4 (IO4); no longer R20.2, U9.8 (IO15)
- net BOOT: now also C25.1; no longer C25.2, C26.1, R19.2
- net DL_RECV: no longer U9.11 (IO18)
- net FL_EMIT: now also U9.38 (IO2); no longer U9.34 (IO41)
- net FL_RECV: now also U9.39 (IO1); no longer U9.10 (IO17)
- net FR_EMIT: now also U9.9 (IO16); no longer U9.35 (IO42)
- net FR_RECV: now also U9.10 (IO17); no longer U9.13 (IO19)
- net GND: now also C22.1, C23.2, C25.2, C26.1, R13.2, C35.2, C36.2, C37.2, C38.2, C39.2, C40.1, C41.2, C42.1, C43.2, C44.2, C45.2, C46.1, C47.1, C48.2, C49.2, C50.2, IC1.4 (GND), IC2.4 (GND), J1.1 (Pin_1), J2.2 (Pin_2), J6.4 (Pin_4), J7.4 (Pin_4), Q12.3 (S), R31.2, R40.2, R46.2, SW3.1, SW4.1, U11.2 (FB), U11.3 (GND), U11.4 (NC), U11.6 (NC), U11.7 (NC), U11.EPAD (GND), U12.4 (SGND), U12.6 (PGND), U12.9 (PAD), U7.2 (FB), U7.3 (GND), U7.4 (NC), U7.6 (NC), U7.7 (NC), U7.EPAD (GND), U8.1 (GND); no longer C22.2, C23.1, C25.1, C26.2, J3.S1 (SHIELD), R15.1, R16.2
- net ML_OUT_A: now also J5.1 (Pin_1)
- net ML_OUT_B: now also J5.2 (Pin_2)
- net ML_PWMA: now also U9.28 (IO35); no longer U9.20 (IO12)
- net ML_PWMB: now also U9.29 (IO36); no longer U9.19 (IO11)
- net MR_OUT_A: now also J4.1 (Pin_1)
- net MR_OUT_B: now also J4.2 (Pin_2)
- net MR_PWMA: now also U9.30 (IO37); no longer U9.24 (IO47)
- net MR_PWMB: now also U9.31 (IO38); no longer U9.23 (IO21)
- net RST: now also C23.1; no longer C23.2
- net SL_RECV: no longer U9.9 (IO16)
- net SR_EMIT: no longer Q8.2 (G), R22.1
- net SR_RECV: now also U9.15 (IO3); no longer U9.14 (IO20)
- net UART_RX: now also J2.3 (Pin_3)
- net UART_TX: now also J2.4 (Pin_4)
- net USB_D+: now also U9.13 (IO19)
- net USB_D-: now also U9.14 (IO20)
- net V_BATTERY: now also C22.2, R20.2, C35.1, C40.2, C47.2, C50.1, J1.2 (Pin_2), U11.8 (VCC), U7.8 (VCC), U8.3 (VI); no longer C15.1, R20.1, U1.7 (P1S/P2S)
- net at R14.2: now also Q12.1 (D)
- net FAN_PWM: now reaches U9.32 (IO39)
- net BTN1: now reaches U9.5 (IO5)
- net BTN1: now also C14.1, SW3.2
- net BTN2: now reaches U9.6 (IO6)
- net BTN2: now also C15.1, SW4.2
- net SDA_0: now reaches U9.7 (IO7)
- net SDA_0: now also R19.1, IC2.6 (SDA), J7.3 (Pin_3), R33.1
- removed net A3.3V: C14.1, C28.1, C29.1, C30.2, U10.13 (VDD), U10.8 (VDDIO)
- net B_BATTERY renamed ML_6V
- net ML_6V: now also U3.6 (VDD), C48.1, U7.1 (Vout)
- net DIAG_EMIT: no longer names the net of U9.33 (IO40)
- net D_EMIT renamed DR_EMIT
- net DR_EMIT: now also U9.11 (IO18)
- net INT: no longer names the net of U10.12 (INT)
- net ML_ENC_A renamed SCL_1
- net SCL_1: now also R16.2, IC1.7 (SCL), J6.2 (Pin_2), R35.1
- net SDI renamed SDA_1
- net SDA_1: now also R15.2, U9.19 (IO11), IC1.6 (SDA), J6.3 (Pin_3), R36.1
- net V_BOOST renamed MR_6V
- net MR_6V: now also U1.7 (P1S/P2S), C49.1, U11.1 (Vout); no longer U3.6 (VDD)
- new net: J3.S1 (SHIELD), R40.1
- new net: R45.1, U12.8 (VREF)
- new net: C43.1, R45.2, R46.1, U12.2 (VCON)
- new net: C37.1, IC2.2 (VDD3V3)
- new net: IC2.8 (DIR), R31.1
- new net: D9.1 (K), R14.1
- new net: C39.1, IC1.2 (VDD3V3)
- new net: IC1.8 (DIR), R34.1
- new net 2V: C44.1, C45.1, D1.2 (A), D2.2 (A), D3.2 (A), D5.2 (A), D6.2 (A), D9.2 (A), U12.3 (FB), U12.5 (VOUT)
- new net DL_EMIT: Q8.2 (G), R22.1, U9.23 (IO21)
- new net SCL_0: IC2.7 (SCL), J7.2 (Pin_2), R28.1, R32.1, U9.8 (IO15)
- new net SL_EMIT: Q12.2 (G), R13.1, U9.20 (IO12)
- new net VBUS: D7.2 (K), D8.2 (A), J3.A4 (VBUS), J3.A9 (VBUS), J3.B4 (VBUS), J3.B9 (VBUS)
- no-connect marks 27 -> 16
Other:
- note added: "6V Motor Regualtors"
- note added: "ESP32 MCU"
- note added: "Encoders"
- note added: "Gyro"
- note added: "USBC"
- moved on the sheet: C10, C11, C12, C13, C19, C20, C21, C23, C25, C28, C29, C30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

Commit message: completed 4 sensor pcb
Parts:
- removed D4: LED, LED_SMD:LED_0805_2012Metric_Pad1.15x1.40mm_HandSolder, symbol Device:LED
- removed R11: R_US, Resistor_SMD:R_0603_1608Metric_Pad0.98x0.95mm_HandSolder, symbol Device:R_US
- added D10: GREEN_LED, LED_SMD:LED_0805_2012Metric_Pad1.15x1.40mm_HandSolder, symbol Device:LED
- added D11: RED_LED, LED_SMD:LED_0805_2012Metric_Pad1.15x1.40mm_HandSolder, symbol Device:LED
- added D12: BLUE_LED, LED_SMD:LED_0805_2012Metric_Pad1.15x1.40mm_HandSolder, symbol Device:LED
- added J8: Conn_01x03_Socket, Connector_PinHeader_2.54mm:PinHeader_1x03_P2.54mm_Vertical, symbol Connector:Conn_01x03_Socket
- added R29, R37: 75, Resistor_SMD:R_0603_1608Metric_Pad0.98x0.95mm_HandSolder, symbol Device:R_US
- added R30: 750, Resistor_SMD:R_0603_1608Metric_Pad0.98x0.95mm_HandSolder, symbol Device:R_US
- C1: value 1uF -> 2.2uF
- J3: footprint Connector_USB:USB_C_Receptacle_GCT_USB4085 -> footprint:CONN16_USB4085-GF-A_GCT
Connections:
- net 3.3V: now also R29.1, R30.1, R37.1
- net 5V: now also J8.3 (Pin_3)
- net FAN_PWM: now also J8.1 (Pin_1)
- net GND: now also J8.2 (Pin_2)
- net RED_LED: now reaches U9.24 (IO47)
- net RED_LED: now also D11.1 (K)
- net BLUE_LED: now reaches U9.25 (IO48)
- net BLUE_LED: now also D12.1 (K)
- net GREEN_LED: now reaches U9.33 (IO40)
- net GREEN_LED: now also D10.1 (K)
- new net: D10.2 (A), R29.2
- new net: D11.2 (A), R30.2
- new net: D12.2 (A), R37.2
Other:
- note added: "LEDs"
- moved on the sheet: J4, J5, R19, R28, U1, U2, U3, U4
