File: pcb_2ir/mercury_2ir.kicad_pcb (KiCad board)
At the start: 2 copper layers, 76 x 99.9 mm, 120 parts, among them J1 Battery, J10 JTAG_Conn2, J2 UART, J3 USB_C_Receptacle_USB2.0, J4 Conn_01x02_Socket, J5 Conn_01x02_Socket, J6 Encoder_L, J7 Encoder_R, J8 Conn_01x03_Socket, J9 JTAG_Conn1, Q1 NMOS, Q2 NMOS, Q3 NMOS, Q4 FR_RECV, Q5 FL_RECV, Q6 R_RECV, Q7 L_RECV, Q8 NMOS, SW1 SW_Push, SW2 SW_Push, SW3 SW_Push, SW4 SW_Push, U1 ZXMHC3F381N8TC, U10 MPU-6500, U12 LMZ10501SILR, U2 UCC27524ADR, U3 UCC27524ADR, U4 ZXMHC3F381N8TC, U5 MCP1700, U6 TPS73633DBV, U8 LM1085-5.0, U9 ESP32-S3-WROOM-1U-N16R8

Commit message: pcb fixes and unit test code for each module of pcb
Parts:
- added D10: POWER_LED, LED_SMD:LED_0805_2012Metric_Pad1.15x1.40mm_HandSolder, F.Cu at (137.7, 84.9)
- added R14: 75, Resistor_SMD:R_0603_1608Metric_Pad0.98x0.95mm_HandSolder, F.Cu at (140.9, 87.9)
- Q1, Q2, Q3, Q8: value NMOS -> Q_NMOS_GSD
- moved C11 3.24 mm to (137.2, 74.6), turned to -135 degrees
- turned C9 to 135 degrees
Connections:
- Q1 pad 1: Net-(Q1-D) -> /FL_EMIT
- Q1 pad 2: /FL_EMIT -> Net-(Q1-S)
- Q2 pad 1: Net-(Q2-D) -> /FR_EMIT
- Q2 pad 2: /FR_EMIT -> Net-(Q2-S)
- Q3 pad 1: Net-(Q3-D) -> /DR_EMIT
- Q3 pad 2: /DR_EMIT -> Net-(Q3-S)
- Q8 pad 1: Net-(Q8-D) -> /DL_EMIT
- Q8 pad 2: /DL_EMIT -> Net-(Q8-S)
- R1 pad 2: Net-(Q1-D) -> Net-(Q1-S)
- R23 pad 2: Net-(Q8-D) -> Net-(Q8-S)
- R3 pad 2: Net-(Q2-D) -> Net-(Q2-S)
- R5 pad 2: Net-(Q3-D) -> Net-(Q3-S)
- U9 pad 13: /USB_D+ -> /USB_D-
- U9 pad 14: /USB_D- -> /USB_D+
Routing:
- net Net-(Q2-S): track 0.00 -> 9.50 mm
- net Net-(Q8-S): track 0.00 -> 7.16 mm
- net /DR_EMIT: track 78.2 -> 82.8 mm, vias 2 -> 4
- net /FL_EMIT: track 76.6 -> 80.5 mm, vias 2 -> 3
- net Net-(Q8-D): track 3.64 -> 0.00 mm
- net Net-(Q1-D): track 3.61 -> 0.00 mm
- net /DL_EMIT: track 72.8 -> 76.1 mm
- net Net-(Q3-S): track 0.00 -> 3.22 mm
- net Net-(Q1-S): track 0.00 -> 2.72 mm
- net 3.3V: track 160.3 -> 162.9 mm
- net Net-(D10-K): track 0.00 -> 2.53 mm
- net Net-(Q2-D): track 2.48 -> 0.00 mm
- net Net-(Q3-D): track 2.43 -> 0.00 mm
- net /USB_D-: track 37.6 -> 36.3 mm
- net Net-(U6-EN): track 11.6 -> 10.6 mm
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Other:
- board text added: "Mercury V2.0 By: Kyle Tyni 2024"
- board text removed: "Mercury_V1 By: Kyle Tyni 2024"
