File: pcb_2ir/mercury_2ir.kicad_sch (KiCad schematic)
At the start: 125 parts, among them IC1 AS5600-ML, IC2 AS5600-MR, J1 Battery, J10 JTAG_Conn2, J2 UART, J3 USB_C_Receptacle_USB2.0, J4 Conn_01x02_Socket, J5 Conn_01x02_Socket, J6 Encoder_L, J7 Encoder_R, J8 Conn_01x03_Socket, J9 JTAG_Conn1, Q1 NMOS, Q2 NMOS, Q3 NMOS, Q4 FR_RECV, Q5 FL_RECV, Q6 R_RECV, Q7 L_RECV, Q8 NMOS, SW1 SW_Push, SW2 SW_Push, SW3 SW_Push, SW4 SW_Push, U1 ZXMHC3F381N8TC, U10 MPU-6500, U12 LMZ10501SILR, U2 UCC27524ADR, U3 UCC27524ADR, U4 ZXMHC3F381N8TC, U5 MCP1700, U6 TPS73633DBV, U8 LM1085-5.0, U9 ESP32-S3-WROOM-1U-N16R8

Commit message: pcb fixes and unit test code for each module of pcb
Parts:
- removed Q1, Q2, Q3, Q8: NMOS, footprint:SOT-23, symbol Simulation_SPICE:NMOS
- added D10: POWER_LED, LED_SMD:LED_0805_2012Metric_Pad1.15x1.40mm_HandSolder, symbol Device:LED
- added Q1, Q2, Q3, Q8: Q_NMOS_GSD, footprint:SOT-23, symbol Device:Q_NMOS_GSD
- added R14: 75, Resistor_SMD:R_0603_1608Metric_Pad0.98x0.95mm_HandSolder, symbol Device:R_US
Connections:
- net 3.3V: now also D10.2 (A)
- net DL_EMIT: now also Q8.1 (G)
- net DR_EMIT: now also Q3.1 (G)
- net FL_EMIT: now also Q1.1 (G)
- net FR_EMIT: now also Q2.1 (G)
- net GND: now also Q1.3 (D), Q2.3 (D), Q3.3 (D), Q8.3 (D), R14.2
- net USB_D+: now also U9.14 (IO20); no longer U9.13 (IO19)
- net USB_D-: now also U9.13 (IO19); no longer U9.14 (IO20)
- net at R5.2: now also Q3.2 (S)
- net at R23.2: now also Q8.2 (S)
- net at R3.2: now also Q2.2 (S)
- net at R1.2: now also Q1.2 (S)
- new net: D10.1 (K), R14.1
