File: main_pcb/main_pcb.kicad_sch (KiCad schematic)
At the start: 127 parts, among them IC1 AS5600-ML, IC2 AS5600-MR, J1 Battery, J10 JTAG_Conn2, J2 UART, J3 USB_C_Receptacle_USB2.0, J4 Conn_01x02_Socket, J5 Conn_01x02_Socket, J6 Encoder_L, J7 Encoder_R, J8 Conn_01x03_Socket, J9 JTAG_Conn1, Q1 Q_NMOS_GSD, Q2 Q_NMOS_GSD, Q3 Q_NMOS_GSD, Q4 FR_RECV, Q5 FL_RECV, Q6 R_RECV, Q7 L_RECV, Q8 Q_NMOS_GSD, SW1 SW_Push, SW2 SW_Push, SW3 SW_Push, SW4 SW_Push, U1 ZXMHC3F381N8TC, U10 MPU-6500, U12 LMZ10501SILR, U2 UCC27524ADR, U3 UCC27524ADR, U4 ZXMHC3F381N8TC, U5 MCP1700, U6 TPS73633DBV, U8 LM1085-5.0, U9 ESP32-S3-WROOM-1U-N16R8

Commit message: cleaned file structure
Other:
- note added: "Mercury V2.1 By: Kyle Tyni 2024"
- moved on the sheet: C14, C15, C19, C20, C21, C23, C25, J10, J2, J6, J7, J8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

Commit message: added basic search implementation
Other:
- note added: "6V Motor Regulators"
- note removed: "6V Motor Regualtors"
Changed lines of the file:
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@@
     (effects (font (size 3.5 3.5)) (justify left bottom))
   )
-  (text "6V Motor Regualtors" (at 306.07 20.32 0)
+  (text "6V Motor Regulators" (at 306.07 20.32 0)
     (effects (font (size 3.5 3.5)) (justify left bottom))
   )
